Commit message: updated generic urdf to match our robot

File: ripl_control/assets/baxter_robot/baxter_description/urdf/baxter.urdf (robot description, URDF)
Before this commit: robot baxter, 57 links, 56 joints
Joints:
- joint left_torso_arm_mount: origin xyz=0.024645 0.219645 0.118588 rpy=0 0 0.7854 -> xyz=0.0250508909425 0.219392814533 0.107748812049 rpy=-0.0074420066736 -0.00129546242287 0.78310045671
- joint right_torso_arm_mount: origin xyz=0.024645 -0.219645 0.118588 rpy=0 0 -0.7854 -> xyz=0.0248817669183 -0.220060922512 0.108693545459 rpy=0.000354590910292 0.00137984354452 -0.780560741676
